File: Kicad/teste/teste.kicad_sch (KiCad schematic)
At the start: 0 parts

Commit message: aulas kicad e vhdl
Parts:
- added U1: ESP32-WROOM-32-GDAE, RF_Module:ESP32-WROOM-32, symbol RF_Module:ESP32-WROOM-32
- added U2: MPU-6050, Sensor_Motion:InvenSense_QFN-24_4x4mm_P0.5mm, symbol Sensor_Motion:MPU-6050
- added U3: BMP280, Package_LGA:Bosch_LGA-8_2x2.5mm_P0.65mm_ClockwisePinNumbering, symbol Sensor_Pressure:BMP280
Connections:
- new net: U1. (3V3), U2.29 (VDD), U3.10 (VDD)
- new net: U1.15 (D15), U1.38 (GND), U1.39 (GND)
- new net 5V: U1. (3V3)
- new net GND: U1. (3V3), U2.28 (GND), U3.9 (GND)
- new net SCL: U1.22 (D22), U2.23 (SCL)
- new net SDA: U1.21 (D21), U2.24 (SDA), U3.3 (SDI)
